Commit message: minor changes

File: yara_description/urdf/yara.urdf (robot description, URDF)
Before this commit: robot yara, 8 links, 7 joints
Links:
- link yara_link_0: geometry collision mesh filename=package://yara_description/meshes/Link0.stl; visual mesh filename=package://yara_description/meshes/Link0.stl
- link yara_link_1: geometry collision mesh filename=package://yara_description/meshes/Link1.stl; visual mesh filename=package://yara_description/meshes/Link1.stl
- link yara_link_2: geometry collision mesh filename=package://yara_description/meshes/Link2.stl; visual mesh filename=package://yara_description/meshes/Link2.stl
- link yara_link_3: geometry collision mesh filename=package://yara_description/meshes/Link3.stl; visual mesh filename=package://yara_description/meshes/Link3.stl
- link yara_link_4: geometry collision mesh filename=package://yara_description/meshes/Link4.stl; visual mesh filename=package://yara_description/meshes/Link4.stl
- link yara_link_5: geometry collision mesh filename=package://yara_description/meshes/Link5.stl; visual mesh filename=package://yara_description/meshes/Link5.stl
